File: Eagle schema/Schema0.1/schema0.1.sch (EAGLE design)
At the start: 17 parts

Commit message: Auto stash before checking out "HEAD"
Parts:
- added BATTERY: B2B-PH-K-S, con-JST PH:B2B-PH-K-S
- added C1: 0.22µF, rcl:C-EUC0805
- added C2: 0.1µF, rcl:C-EUC0805
- added C3: 10µF, rcl:CPOL-EUE2-5
- added C4: 10µ, rcl:CPOL-EUE2-5
- added IC1: 7805T, adafruit:7805T
- added LM1117: 317EMP, linear:317EMP
- added MHZ19: B7B-PH-KL, con-JST PH:B7B-PH-KL
- CJMCU-811: value (none) -> B8B-PH-K-S; device con-lstb:MA08-1 -> con-JST PH:B8B-PH-K-S
- DHT22, MQ-135, MQ-7, SDS011, SV1: value (none) -> B4B-PH-K-S; device con-lstb:MA04-1 -> con-JST PH:B4B-PH-K-S
- LM35: value (none) -> B3B-PH-KL; device con-lstb:MA03-1 -> con-JST PH:B3B-PH-KL
- R1, R2, R3, R5, R6, R7, R8, R9: device rcl:R-EU_0207/10 -> rcl:R-EU_R0805
Connections:
- new net AMHZ19: MHZ19.1, U$2.IO33
- new net RX2: MHZ19.5, U$2.IO19
- new net TX2: MHZ19.6, U$2.IO18
- new net VIN: BATTERY.1, C1.1, C4.+, IC1.VI, LM1117.VI
- net 3.3V: now also C3.+, LM1117.VO
- net 5V: now also C2.1, IC1.VO, MHZ19.4
- net GND: now also BATTERY.2, C1.2, C2.2, C3.-, C4.-, IC1.GND, LM1117.ADJ, MHZ19.3
Other:
- note added: "Air Quality Sensor"
